File: DLSB-DRIVERBOARD-V1.kicad_sch (KiCad schematic)
At the start: 14 parts, among them J1 HEAD-I01-X-PI2X03-SM-H2X3SM, J2 HEAD-I01-X-PI2X03-SM-H2X3SM, Q1 TRNN-SO23-X-KS8050-01-TRNN-SO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, Q2 MOSN-T252-X-K4184-01-MN252418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, U1 MCUU-SC14-84-ATTINY-01-MCAT84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, U2 VREG-SO223-X-KLD1117-V33D-VR1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, Y1 XTAL-5032-X-MZ16-01-XTAL5032-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

Commit message: First PCB order.
Parts:
- added J3: HEAD-JSTSH-X-PI04-RS-HSH04RS, oomlout_OOMP_parts:HEAD-JSTSH-X-PI04-RS-HSH04RS, symbol oomlout_OOMP_parts:HEAD-JSTSH-X-PI04-RS-HSH04RS
- added J4: HEAD-I01-X-PI01-01-HP01, oomlout_OOMP_parts:HEAD-I01-X-PI01-01-HP01, symbol oomlout_OOMP_parts:HEAD-I01-X-PI01-01-HP01
Connections:
- net SCK is gone; now on net ADC4: J1.3 (Pin_3)
- net ADC0: now also J4.1 (Pin_1)
- net ADC4: now also J3.4 (Pin_4)
- net ADC6: now also J3.3 (Pin_3)
- net GND: now also J3.1 (Pin_1)
- net VCC: now also J3.2 (Pin_2)
Other:
- note added: "MODULE-CONN I2C-QWIIC-01 oom.lt/MCQ"
